File: kicad/board/_autosave-board.kicad_pcb (KiCad board)
At the start: 4 copper layers, 58.7 x 74.9 mm, 59 parts, among them J1 i2c_connector, J2 uart_connector, J3 spi_connector, J4 debug header, J5 powerheader, J6 USB_B_Micro, J7 gpioheader A, J8 gpioheader B, SW1 reset button, SW2 pw_sw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

Commit message: v1.1 adding
Routing:
- net GND: vias 20 -> 24
