File: kicad/board/board.sch (KiCad schematic (older format))
At the start: 45 parts, among them J1 i2c_connector, J2 uart_connector, J3 spi_connector, J4 debug header, J5 powerheader, J6 USB_B_Micro, J7 gpioheader A, J8 gpioheader B, SW1 reset button, U1 BQ24075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

Commit message: v1.1 adding
Parts:
- added D2: red_led, LED_SMD:LED_0603_1608Metric, symbol Device:LED_Small
- added D3: green_led, LED_SMD:LED_0603_1608Metric, symbol Device:LED_Small
- added R11: 3.0K, Resistor_SMD:R_0603_1608Metric_Pad0.98x0.95mm_HandSolder, symbol Device:R_Small
- added R12: 150, Resistor_SMD:R_0402_1005Metric, symbol Device:R_Small
- added R13: 100, Resistor_SMD:R_0402_1005Metric, symbol Device:R_Small
- added R14, R15: 10kΩ, Resistor_SMD:R_0402_1005Metric, symbol Device:R_Small
- added SW2: pw_sw, components:K301235D, symbol Switch:SW_SPDT
- added TP3: batvoltage, TestPoint:TestPoint_Pad_D1.0mm, symbol Connector:TestPoint
- BT1: lcsc C152154 -> (none)
- C1, C2: lcsc C26408 -> (none)
- C10, C3, C8: lcsc C19666 -> (none)
- C11: lcsc C57112 -> (none)
- C12, C13, C4: lcsc C1848 -> (none)
- C14, C5, C6, C7, C9: lcsc C1525 -> (none)
- D1: lcsc C108793 -> (none)
- J1: lcsc C124378 -> (none)
- J2: LCSC C492414 -> C225514; lcsc C492414 -> (none)
- J3: lcsc C492405 -> (none)
- J4: lcsc C5665 -> (none)
- J5: lcsc C124381 -> (none)
- J6: lcsc C132563 -> (none)
- JP1, JP2: lcsc C49257 -> (none)
- R1: value 1.13kΩ -> 1.8kΩ; footprint Resistor_SMD:R_0402_1005Metric -> Resistor_SMD:R_0603_1608Metric_Pad0.98x0.95mm_HandSolder; LCSC C67014 -> C4177; lcsc C67014 -> (none)
- R10, R8: pick&placed (none) -> YES
- R2: lcsc C25744 -> (none)
- R3: lcsc C25131 -> (none)
- R4, R5: lcsc C25083 -> (none)
- R6: LCSC C98835 -> C98835
- R7, R9: LCSC C25900 -> C25900; pick&placed (none) -> YES
- SW1: lcsc C223748 -> (none)
- TP1, TP2: footprint TestPoint:TestPoint_Pad_D2.0mm -> TestPoint:TestPoint_Pad_D1.0mm
- U1: lcsc C15464 -> (none)
- U2: lcsc C8304 -> (none)
- U3: lcsc C80670 -> (none)
- U4: lcsc C81195 -> (none)
- Y1: lcsc C13738 -> (none)
Connections:
- net +3V3: now also J7.12 (Pin_12)
- net +5V: now also D2.2 (A), D3.2 (A)
- net GND: now also J7.14 (Pin_14), R11.2, SW2.1 (A)
- net RGB_B: now also J5.1 (Pin_1); no longer J5.3 (Pin_3)
- net RGB_G: now also J5.3 (Pin_3); no longer J5.1 (Pin_1)
- net boot0: now also R14.2; no longer JP1.2
- net boot1: now also J8.11 (Pin_11), R15.2; no longer J7.15 (Pin_15), JP2.2
- net eeprom_scl: now also J8.13 (Pin_13); no longer J7.13 (Pin_13)
- net eeprom_sda: now also J8.15 (Pin_15); no longer J7.11 (Pin_11)
- net i2c_scl: now also J8.14 (Pin_14); no longer J8.15 (Pin_15)
- net i2c_sda: now also J8.12 (Pin_12); no longer J8.13 (Pin_13)
- net pa0: now also J8.10 (Pin_10); no longer J7.16 (Pin_16)
- net pa1: now also J8.8 (Pin_8); no longer J7.14 (Pin_14)
- net pa15: now also J7.7 (Pin_7); no longer J8.2 (Pin_2)
- net pa2: now also J8.6 (Pin_6); no longer J7.12 (Pin_12)
- net pa3: now also J8.4 (Pin_4); no longer J7.10 (Pin_10)
- net pa8: now also J7.6 (Pin_6); no longer J8.11 (Pin_11)
- net pb0: now also J8.7 (Pin_7); no longer J7.1 (Pin_1)
- net pb1: now also J8.9 (Pin_9); no longer J7.3 (Pin_3)
- net pb12: now also J7.3 (Pin_3); no longer J7.9 (Pin_9)
- net pb13: now also J7.1 (Pin_1); no longer J7.7 (Pin_7)
- net pb14: now also J7.2 (Pin_2); no longer J7.5 (Pin_5)
- net pb15: now also J7.4 (Pin_4); no longer J8.16 (Pin_16)
- net pb3: now also J7.9 (Pin_9); no longer J8.1 (Pin_1)
- net pb4: now also J7.11 (Pin_11); no longer J8.3 (Pin_3)
- net pb5: now also J7.13 (Pin_13); no longer J8.5 (Pin_5)
- net pb6: now also J7.15 (Pin_15); no longer J8.7 (Pin_7)
- net pb7: now also J8.16 (Pin_16); no longer J8.9 (Pin_9)
- net spi_cs: now also J3.1 (Pin_1), J8.2 (Pin_2); no longer J3.4 (Pin_4), J7.8 (Pin_8)
- net spi_miso: now also J8.3 (Pin_3); no longer J7.4 (Pin_4)
- net spi_mosi: now also J3.4 (Pin_4), J8.5 (Pin_5); no longer J3.2 (Pin_2), J7.2 (Pin_2)
- net spi_sclk: now also J3.2 (Pin_2), J8.1 (Pin_1); no longer J3.1 (Pin_1), J7.6 (Pin_6)
- net swclk: now also J7.5 (Pin_5); no longer J8.4 (Pin_4)
- net swdio: now also J7.16 (Pin_16); no longer J8.6 (Pin_6)
- net uart_rx: now also J7.10 (Pin_10); no longer J8.12 (Pin_12)
- net uart_tx: now also J7.8 (Pin_8); no longer J8.14 (Pin_14)
- net usb_d+: no longer J8.8 (Pin_8)
- net usb_d-: no longer J8.10 (Pin_10)
- net at C12.2, C8.2, JP3.2 (B)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: now also SW2.3 (C); no longer U3.3 (EN)
- net at U1.12 (ILIM): now also R11.1
- net at BT1.1 (+), C10.1, U1.2 (BAT)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: now also TP3.1
- net at U1.7 (~PGOOD): now also R13.1
- net at U1.9 (~CHG): now also R12.2
- new net: JP1.2, R14.1
- new net: JP2.2, R15.1
- new net: SW2.2 (B), U3.3 (EN)
- new net: D2.1 (K), R12.1
- new net: D3.1 (K), R13.2
- no-connect marks 8 -> 4
Other:
- moved on the sheet: BT1, C10, C12, C13, C4, C8, JP3, R1, R2, TP1, TP2, U1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

Commit message: putting the thermistor replacement resistor to gnd instead of 5v fixing #18
Connections:
- net +5V: no longer R2.2
- net GND: now also R2.2
Changed lines of the file:
@@
-$EndComp
-$Comp
-L power:+5V #PWR018
-U 1 1 5F64035F
-P 2500 6775
-F 0 "#PWR018" H 2500 6625 50  0001 C CNN
-F 1 "+5V" H 2515 6948 50  0000 C CNN
-F 2 "" H 2500 6775 50  0001 C CNN
-F 3 "" H 2500 6775 50  0001 C CNN
-	1    2500 6775
-	-1   0    0    1
 $EndComp
 $Comp
@@
 	1    0    0    -1
 $EndComp
+$Comp
+L power:GND #PWR?
+U 1 1 5FFB8250
+P 2500 6775
+F 0 "#PWR?" H 2500 6525 50  0001 C CNN
+F 1 "GND" H 2505 6602 50  0000 C CNN
+F 2 "" H 2500 6775 50  0001 C CNN
+F 3 "" H 2500 6775 50  0001 C CNN
+	1    2500 6775
+	1    0    0    -1
+$EndComp

Commit message: adding testpoint to measure bat charge current This will make it easier to identify bat charging problems.
Parts:
- added TP4: batcurrent, TestPoint:TestPoint_Pad_D1.0mm, symbol Connector:TestPoint
Connections:
- net at R1.2, U1.16 (ISET): now also TP4.1
Other:
- moved on the sheet: R1

Commit message: changing crystal for a 8MHz one instead of 16MHz
Parts:
- removed Y1: X322516MLB4SI, components:YSX321SL, symbol Device:Crystal_GND24_Small
- added Y1: X50328MSB2GI, Crystal:Crystal_SMD_5032-2Pin_5.0x3.2mm, symbol Device:Crystal
- C1, C2: value 8pF -> 30pF; LCSC C26408 -> C1570
Connections:
- net at C1.1, U2.5 (PD0): now also Y1.1
- net at C2.1, U2.6 (PD1): now also Y1.2
Changed lines of the file:
@@
 P 1100 1950
 F 0 "C1" V 871 1950 50  0000 C CNN
-F 1 "8pF" V 962 1950 50  0000 C CNN
+F 1 "30pF" V 962 1950 50  0000 C CNN
 F 2 "Capacitor_SMD:C_0402_1005Metric" H 1100 1950 50  0001 C CNN
 F 3 "https://datasheet.lcsc.com/szlcsc/1809301912_YAGEO-CC0402JRNPO9BN220_C106203.pdf" H 1100 1950 50  0001 C CNN
 F 4 "" H 1100 1950 50  0001 C CNN "lcsc"
 F 5 "YES" H 1100 1950 50  0001 C CNN "pick&placed"
-F 6 "C26408" H 1100 1950 50  0001 C CNN "LCSC"
+F 6 "C1570" H 1100 1950 50  0001 C CNN "LCSC"
 	1    1100 1950
 	0    1    1    0
@@
 P 1100 2250
 F 0 "C2" V 1300 2250 50  0000 C CNN
-F 1 "8pF" V 1200 2250 50  0000 C CNN
+F 1 "30pF" V 1200 2250 50  0000 C CNN
 F 2 "Capacitor_SMD:C_0402_1005Metric" H 1100 2250 50  0001 C CNN
 F 3 "https://datasheet.lcsc.com/szlcsc/1809301912_YAGEO-CC0402JRNPO9BN220_C106203.pdf" H 1100 2250 50  0001 C CNN
 F 4 "" H 1100 2250 50  0001 C CNN "lcsc"
 F 5 "YES" H 1100 2250 50  0001 C CNN "pick&placed"
-F 6 "C26408" H 1100 2250 50  0001 C CNN "LCSC"
+F 6 "C1570" H 1100 2250 50  0001 C CNN "LCSC"
 	1    1100 2250
 	0    1    1    0
@@
 Wire Wire Line
 	4375 6325 4475 6325
-Wire Wire Line
-	1200 2250 1300 2250
-Wire Wire Line
-	1200 1950 1300 1950
-$Comp
-L Device:Crystal_GND24_Small Y1
-U 1 1 5F9BF43B
-P 1300 2100
-F 0 "Y1" V 1100 2000 50  0000 L CNN
-F 1 "X322516MLB4SI" V 1250 1300 50  0000 L CNN
-F 2 "components:YSX321SL" H 1300 2100 50  0001 C CNN
-F 3 "~" H 1300 2100 50  0001 C CNN
-F 4 "" H 1300 2100 50  0001 C CNN "lcsc"
-F 5 "YES" H 1300 2100 50  0001 C CNN "pick&placed"
-F 6 "C13738" H 1300 2100 50  0001 C CNN "LCSC"
-	1    1300 2100
-	0    1    1    0
-$EndComp
-Wire Wire Line
-	1300 2000 1300 1950
-Connection ~ 1300 1950
-Wire Wire Line
-	1300 1950 1500 1950
-Wire Wire Line
-	1300 2200 1300 2250
-Connection ~ 1300 2250
-Wire Wire Line
-	1300 2250 1500 2250
-$Comp
-L power:GND #PWR0102
-U 1 1 5F9C6A9D
-P 1400 2100
-F 0 "#PWR0102" H 1400 1850 50  0001 C CNN
-F 1 "GND" V 1500 2175 50  0000 R CNN
-F 2 "" H 1400 2100 50  0001 C CNN
-F 3 "" H 1400 2100 50  0001 C CNN
-	1    1400 2100
-	0    -1   -1   0
-$EndComp
-$Comp
-L power:GND #PWR0103
-U 1 1 5F9C7055
-P 1200 2100
-F 0 "#PWR0103" H 1200 1850 50  0001 C CNN
-F 1 "GND" V 1250 1950 50  0000 R CNN
-F 2 "" H 1200 2100 50  0001 C CNN
-F 3 "" H 1200 2100 50  0001 C CNN
-	1    1200 2100
-	0    1    1    0
-$EndComp
 $Comp
 L Device:R_Small R7
@@
 Wire Wire Line
 	1025 7000 1025 7025
+Wire Wire Line
+	1200 1950 1300 1950
+Wire Wire Line
+	1200 2250 1300 2250
+$Comp
+L Device:Crystal Y1
+U 1 1 6003A965
+P 1300 2100
+F 0 "Y1" V 1200 2025 50  0000 R CNN
+F 1 "X50328MSB2GI" V 1300 2800 50  0000 R CNN
+F 2 "Crystal:Crystal_SMD_5032-2Pin_5.0x3.2mm" H 1300 2100 50  0001 C CNN
+F 3 "https://datasheet.lcsc.com/szlcsc/1903061615_Yangxing-Tech-X50328MSB2GI_C115962.pdf" H 1300 2100 50  0001 C CNN
+F 4 " C115962" V 1300 2100 50  0001 C CNN "LCSC"
+	1    1300 2100
+	0    -1   1    0
+$EndComp
+Connection ~ 1300 2250
+Wire Wire Line
+	1300 2250 1500 2250
+Connection ~ 1300 1950
+Wire Wire Line
+	1300 1950 1500 1950
 $EndSCHEMATC

Commit message: making the leds less bright by replacing r12 and r13 for 1k fixing #16
Parts:
- R12: value 150 -> 1k; LCSC C25082 -> C11702
- R13: value 100 -> 1k; LCSC C25076 -> C11702
Changed lines of the file:
@@
 P 2375 7125
 F 0 "R13" H 2575 7150 50  0000 R CNN
-F 1 "100" H 2575 7075 50  0000 R CNN
+F 1 "1k" H 2575 7075 50  0000 R CNN
 F 2 "Resistor_SMD:R_0402_1005Metric" H 2375 7125 50  0001 C CNN
 F 3 "~" H 2375 7125 50  0001 C CNN
-F 4 "C25076" H 2375 7125 50  0001 C CNN "LCSC"
+F 4 "C11702" H 2375 7125 50  0001 C CNN "LCSC"
 F 5 "YES" H 2375 7125 50  0001 C CNN "pick&placed"
 	1    2375 7125
@@
 P 2225 7125
 F 0 "R12" H 2425 7100 50  0000 R CNN
-F 1 "150" H 2425 7175 50  0000 R CNN
+F 1 "1k" H 2425 7175 50  0000 R CNN
 F 2 "Resistor_SMD:R_0402_1005Metric" H 2225 7125 50  0001 C CNN
 F 3 "https://datasheet.lcsc.com/szlcsc/Hubei-KENTO-Elec-KT-0603R_C2286.pdf" H 2225 7125 50  0001 C CNN
-F 4 "C25082" H 2225 7125 50  0001 C CNN "LCSC"
+F 4 "C11702" H 2225 7125 50  0001 C CNN "LCSC"
 F 5 "YES" H 2225 7125 50  0001 C CNN "pick&placed"
 	1    2225 7125
